Commit message: need to get the frame prefix figured out

File: nuturtle_description/urdf/turtlebot3_burger.urdf.xacro (robot description, xacro)
@@ -1,6 +1,4 @@
 <?xml version="1.0" ?>
 <robot name="turtlebot3_burger" xmlns:xacro="http://ros.org/wiki/xacro">
-  <!-- <xacro:include filename="$(find nuturtle_description)/urdf/common_properties.xacro"/>
-  <xacro:include filename="$(find nuturtle_description)/urdf/turtlebot3_burger.gazebo.xacro"/> -->
   <xacro:property name="bot_params" value="$(find nuturtle_description)/config/diff_params.yaml" />
   <xacro:property name="params" value="${xacro.load_yaml(bot_params)['/**']['ros__parameters']}" />
@@ -8,4 +6,5 @@
   <xacro:property name="track_width"  value="${params['track_width']}" />
   <xacro:property name="collision_radius"  value="${params['collision_radius']}" />
+  <xacro:arg name="color"  default="purple" />
   <material name="black">
     <color rgba="0.0 0.0 0.0 1.0"/>
@@ -23,15 +22,9 @@
     <color rgba="0.0 0.8 0.0 1.0"/>
   </material>
-  <material name="grey">
-    <color rgba="0.5 0.5 0.5 1.0"/>
-  </material>
-  <material name="orange">
-    <color rgba="${255/255} ${108/255} ${10/255} 1.0"/>
-  </material>
-  <material name="brown">
-    <color rgba="${222/255} ${207/255} ${195/255} 1.0"/>
-  </material>
   <material name="red">
     <color rgba="0.8 0.0 0.0 1.0"/>
+  </material>
+  <material name="purple">
+    <color rgba="0.3 0.16 0.52 1.0"/>
   </material>
   <material name="white">
@@ -50,5 +43,5 @@
         <mesh filename="package://nuturtle_description/meshes/burger_base.stl" scale="0.001 0.001 0.001"/>
       </geometry>
-      <material name="light_black"/>
+      <material name="$(arg color)"/>
     </visual>
     <xacro:if value = "${collision_radius>=0}">
